Commit message: work on gripper urdf

File: ur3e_moveit_config/urdf/inc/ur_macro.xacro (robot description, xacro)
@@ -42,6 +42,6 @@
      - Muhammad Asif Rana
   -->
-  <xacro:include filename="$(find ur_description)/urdf/inc/ur_transmissions.xacro" />
-  <xacro:include filename="$(find ur_description)/urdf/inc/ur_common.xacro" />
+  <xacro:include filename="$(find ur3e_moveit_config)/urdf/inc/ur_transmissions.xacro" />
+  <xacro:include filename="$(find ur3e_moveit_config)/urdf/inc/ur_common.xacro" />
   <xacro:macro name="ur_robot" params="
     prefix
@@ -316,10 +316,9 @@
       <child link="${prefix}tool0"/>
     </joint>
-    <!-- Define the end effector link -->
     <link name="end_effector_link">
       <visual>
-        <!-- Define visual properties (e.g., geometry, color) -->
-        <geometry>
-          <box size="0.05 0.05 0.05"/> <!-- Example: a small cube -->
+        <origin xyz="0 0 0" rpy="0 0 0"/>
+        <geometry>
+          <mesh filename="package://ur3e_moveit_config/meshes/ur3e/collision/gripper_stl.stl"/> <!-- Replace path/to/end_effector.stl with the actual path -->
         </geometry>
         <material name="end_effector_material">
@@ -328,14 +327,13 @@
       </visual>
       <collision>
-        <!-- Define collision properties (e.g., simplified geometry) -->
-        <geometry>
-          <box size="0.05 0.05 0.05"/> <!-- Example: same size as visual -->
-        </geometry>
-      </collision>
-      <!-- Define inertia properties (e.g., mass, moments of inertia) -->
+        <origin xyz="0 0 0" rpy="0 0 0"/>
+        <geometry>
+          <mesh filename="package://ur3e_moveit_config/meshes/ur3e/collision/gripper_stl.stl"/> <!-- Same mesh file used for collision -->
+        </geometry>
+      </collision>
       <inertial>
-        <mass value="0.1"/> <!-- Example: mass of 0.1 kg -->
+        <mass value="0.5"/> <!-- Example: mass of 1.0 kg -->
         <!-- Define the inertia matrix -->
-        <inertia ixx="0.001" iyy="0.001" izz="0.001" ixy="0" ixz="0" iyz="0"/>
+        <inertia ixx="0.1" iyy="0.1" izz="0.1" ixy="0" ixz="0" iyz="0"/>
       </inertial>
     </link>

Commit message: end effector added need more states

File: ur3e_moveit_config/urdf/inc/ur_macro.xacro (robot description, xacro)
@@ -318,16 +318,16 @@
     <link name="end_effector_link">
       <visual>
-        <origin xyz="0 0 0" rpy="0 0 0"/>
-        <geometry>
-          <mesh filename="package://ur3e_moveit_config/meshes/ur3e/collision/gripper_stl.stl"/> <!-- Replace path/to/end_effector.stl with the actual path -->
+        <origin xyz="-0.079 0.032 0.0738" rpy="0 -3.141592653589793 3.141592653589793"/>
+        <geometry>
+          <mesh filename="package://ur3e_moveit_config/meshes/ur3e/collision/gripper.stl"/> <!-- Replace path/to/end_effector.stl with the actual path -->
         </geometry>
         <material name="end_effector_material">
-          <color rgba="0.5 0.5 0.5 1"/> <!-- Example: light gray color -->
-        </material>
-      </visual>
-      <collision>
-        <origin xyz="0 0 0" rpy="0 0 0"/>
-        <geometry>
-          <mesh filename="package://ur3e_moveit_config/meshes/ur3e/collision/gripper_stl.stl"/> <!-- Same mesh file used for collision -->
+          <color rgba="0.4901961 0.6784314 0.8 1"/> <!-- Example: light gray color -->
+        </material>
+      </visual>
+      <collision>
+        <origin xyz="-0.079 0.032 0.0738" rpy="0 -3.141592653589793 3.141592653589793"/>
+        <geometry>
+          <mesh filename="package://ur3e_moveit_config/meshes/ur3e/collision/gripper.stl"/> <!-- Same mesh file used for collision -->
         </geometry>
       </collision>

Commit message: Cartesian point works

File: ur3e_moveit_config/urdf/inc/ur_macro.xacro (robot description, xacro)
@@ -318,5 +318,5 @@
     <link name="end_effector_link">
       <visual>
-        <origin xyz="-0.079 0.032 0.0738" rpy="0 -3.141592653589793 3.141592653589793"/>
+        <origin xyz="-0.079 0.032 -0.0462" rpy="0 -3.141592653589793 3.141592653589793"/>
         <geometry>
           <mesh filename="package://ur3e_moveit_config/meshes/ur3e/collision/gripper.stl"/> <!-- Replace path/to/end_effector.stl with the actual path -->
@@ -327,5 +327,5 @@
       </visual>
       <collision>
-        <origin xyz="-0.079 0.032 0.0738" rpy="0 -3.141592653589793 3.141592653589793"/>
+        <origin xyz="-0.079 0.032 -0.0462" rpy="0 -3.141592653589793 3.141592653589793"/>
         <geometry>
           <mesh filename="package://ur3e_moveit_config/meshes/ur3e/collision/gripper.stl"/> <!-- Same mesh file used for collision -->
@@ -343,5 +343,5 @@
       <child link="end_effector_link"/>
       <!-- Define the transformation from the last link to the end effector -->
-      <origin xyz="0 0 0.1" rpy="0 0 0"/> <!-- Example: 0.1 meter offset in the z-axis -->
+      <origin xyz="0 0 0.22" rpy="0 0 0"/> <!-- Example: 0.1 meter offset in the z-axis -->
     </joint>
   </xacro:macro>

Commit message: work on setup env function

File: ur3e_moveit_config/urdf/inc/ur_macro.xacro (robot description, xacro)
@@ -345,4 +345,16 @@
       <origin xyz="0 0 0.22" rpy="0 0 0"/> <!-- Example: 0.1 meter offset in the z-axis -->
     </joint>
+    <!-- Define the camera link -->
+    <link name="camera_frame">
+      <!-- Define the visual and collision properties of the camera -->
+      <!-- Add visual and collision elements here -->
+    </link>
+    <!-- Connect the camera frame to an existing link on the robot -->
+    <joint name="camera_joint" type="fixed">
+      <parent link="end_effector_link"/>
+      <child link="camera_frame"/>
+      <!-- Specify the transformation between the camera frame and the parent link -->
+      <origin xyz="0 -0.065 -0.15" rpy="-0.31416 0 0"/>
+    </joint>
   </xacro:macro>
 </robot>

Commit message: works on robot next button task

File: ur3e_moveit_config/urdf/inc/ur_macro.xacro (robot description, xacro)
@@ -355,5 +355,5 @@
       <child link="camera_frame"/>
       <!-- Specify the transformation between the camera frame and the parent link -->
-      <origin xyz="0 -0.065 -0.15" rpy="-0.31416 0 0"/>
+      <origin xyz="0 -0.065 -0.15" rpy="-0.2967059728 -0.0261799388 0"/>
     </joint>
   </xacro:macro>

Commit message: IMU task in work

File: ur3e_moveit_config/urdf/inc/ur_macro.xacro (robot description, xacro)
@@ -320,5 +320,5 @@
         <origin xyz="-0.079 0.032 -0.0462" rpy="0 -3.141592653589793 3.141592653589793"/>
         <geometry>
-          <mesh filename="package://ur3e_moveit_config/meshes/ur3e/collision/gripper.stl"/> <!-- Replace path/to/end_effector.stl with the actual path -->
+          <mesh filename="package://ur3e_moveit_config/meshes/ur3e/collision/full_assembly_part_open.stl"/> <!-- Replace path/to/end_effector.stl with the actual path -->
         </geometry>
         <material name="end_effector_material">
@@ -329,5 +329,5 @@
         <origin xyz="-0.079 0.032 -0.0462" rpy="0 -3.141592653589793 3.141592653589793"/>
         <geometry>
-          <mesh filename="package://ur3e_moveit_config/meshes/ur3e/collision/gripper.stl"/> <!-- Same mesh file used for collision -->
+          <mesh filename="package://ur3e_moveit_config/meshes/ur3e/collision/full_assembly_part_open.stl"/> <!-- Same mesh file used for collision -->
         </geometry>
       </collision>

Commit message: Works now work on kinematic

File: ur3e_moveit_config/urdf/inc/ur_macro.xacro (robot description, xacro)
@@ -320,5 +320,5 @@
         <origin xyz="-0.079 0.032 -0.0462" rpy="0 -3.141592653589793 3.141592653589793"/>
         <geometry>
-          <mesh filename="package://ur3e_moveit_config/meshes/ur3e/collision/full_assembly_part_open.stl"/> <!-- Replace path/to/end_effector.stl with the actual path -->
+          <mesh filename="package://ur3e_moveit_config/meshes/ur3e/collision/full_assembly_part_v2_added_more_to_camera.stl"/> <!-- Replace path/to/end_effector.stl with the actual path -->
         </geometry>
         <material name="end_effector_material">
@@ -329,5 +329,5 @@
         <origin xyz="-0.079 0.032 -0.0462" rpy="0 -3.141592653589793 3.141592653589793"/>
         <geometry>
-          <mesh filename="package://ur3e_moveit_config/meshes/ur3e/collision/full_assembly_part_open.stl"/> <!-- Same mesh file used for collision -->
+          <mesh filename="package://ur3e_moveit_config/meshes/ur3e/collision/full_assembly_part_v2_added_more_to_camera.stl"/> <!-- Same mesh file used for collision -->
         </geometry>
       </collision>

Commit message: small changes

File: ur3e_moveit_config/urdf/inc/ur_macro.xacro (robot description, xacro)
@@ -320,5 +320,5 @@
         <origin xyz="-0.079 0.032 -0.0462" rpy="0 -3.141592653589793 3.141592653589793"/>
         <geometry>
-          <mesh filename="package://ur3e_moveit_config/meshes/ur3e/collision/full_assembly_part_v2_added_more_to_camera.stl"/> <!-- Replace path/to/end_effector.stl with the actual path -->
+          <mesh filename="package://ur3e_moveit_config/meshes/ur3e/collision/full_assembly_part_v3.stl"/> <!-- Replace path/to/end_effector.stl with the actual path -->
         </geometry>
         <material name="end_effector_material">
@@ -329,5 +329,5 @@
         <origin xyz="-0.079 0.032 -0.0462" rpy="0 -3.141592653589793 3.141592653589793"/>
         <geometry>
-          <mesh filename="package://ur3e_moveit_config/meshes/ur3e/collision/full_assembly_part_v2_added_more_to_camera.stl"/> <!-- Same mesh file used for collision -->
+          <mesh filename="package://ur3e_moveit_config/meshes/ur3e/collision/full_assembly_part_v3.stl"/> <!-- Same mesh file used for collision -->
         </geometry>
       </collision>

Commit message: OMPL test done

File: ur3e_moveit_config/urdf/inc/ur_macro.xacro (robot description, xacro)
@@ -316,45 +316,4 @@
       <child link="${prefix}tool0"/>
     </joint>
-    <link name="end_effector_link">
-      <visual>
-        <origin xyz="-0.079 0.032 -0.0462" rpy="0 -3.141592653589793 3.141592653589793"/>
-        <geometry>
-          <mesh filename="package://ur3e_moveit_config/meshes/ur3e/collision/full_assembly_part_v3.stl"/> <!-- Replace path/to/end_effector.stl with the actual path -->
-        </geometry>
-        <material name="end_effector_material">
-          <color rgba="0.4901961 0.6784314 0.8 1"/> <!-- Example: light gray color -->
-        </material>
-      </visual>
-      <collision>
-        <origin xyz="-0.079 0.032 -0.0462" rpy="0 -3.141592653589793 3.141592653589793"/>
-        <geometry>
-          <mesh filename="package://ur3e_moveit_config/meshes/ur3e/collision/full_assembly_part_v3.stl"/> <!-- Same mesh file used for collision -->
-        </geometry>
-      </collision>
-      <inertial>
-        <mass value="0.5"/> <!-- Example: mass of 1.0 kg -->
-        <!-- Define the inertia matrix -->
-        <inertia ixx="0.1" iyy="0.1" izz="0.1" ixy="0" ixz="0" iyz="0"/>
-      </inertial>
-    </link>
-    <!-- Connect the end effector to the last link of the robot arm -->
-    <joint name="end_effector_joint" type="fixed">
-      <parent link="tool0"/> <!-- Adjust link name accordingly -->
-      <child link="end_effector_link"/>
-      <!-- Define the transformation from the last link to the end effector -->
-      <origin xyz="0 0 0.22" rpy="0 0 0"/> <!-- Example: 0.1 meter offset in the z-axis -->
-    </joint>
-    <!-- Define the camera link -->
-    <link name="camera_frame">
-      <!-- Define the visual and collision properties of the camera -->
-      <!-- Add visual and collision elements here -->
-    </link>
-    <!-- Connect the camera frame to an existing link on the robot -->
-    <joint name="camera_joint" type="fixed">
-      <parent link="end_effector_link"/>
-      <child link="camera_frame"/>
-      <!-- Specify the transformation between the camera frame and the parent link -->
-      <origin xyz="0 -0.065 -0.15" rpy="-0.2967059728 -0.0261799388 0"/>
-    </joint>
   </xacro:macro>
 </robot>
